Commit message: Fixed issue with controller_manager not starting by remapping the robot_description topic the manager listens on

File: src/terrestrial_robot/description/urdf/Terrestrial_Robot_Export.xacro (robot description, xacro)
@@ -5,9 +5,9 @@
 <xacro:include filename="$(find Terrestrial_Robot_Export_description)/urdf/Terrestrial_Robot_Export.gazebo" />
 <link name="base_link">
-  <inertial>
+  <!-- <inertial>
     <origin xyz="-5.183336997375715e-17 -0.007592361577329013 0.006868005732278094" rpy="0 0 0"/>
     <mass value="4.133882166278983"/>
     <inertia ixx="0.015635" iyy="0.018694" izz="0.033526" ixy="0.0" iyz="0.000385" ixz="-0.0"/>
-  </inertial>
+  </inertial> -->
   <visual>
     <origin xyz="0 0 0" rpy="0 0 0"/>
@@ -228,4 +228,3 @@
   <axis xyz="1.0 0.0 0.0"/>
 </joint>
-<xacro:include filename="$(find Terrestrial_Robot_Export_description)/urdf/gazebo_config.xacro" />
 </robot>
