Commit message: Separated sim xacro logic from real stuff because of GazeboSystem vs Actuator types

File: src/terrestrial_robot/description/urdf/ros2_control_config.xacro (robot description, xacro)
@@ -2,89 +2,114 @@
 <robot name="Terrestrial Robot" xmlns:xacro="http://www.ros.org/wiki/xacro" >
 <xacro:macro name="terrestrial_robot_ros2_control" params="simulation fr_label fl_label br_label bl_label">
-<ros2_control name="Actuator_${bl_label}" type="actuator">
-  <xacro:if value="${simulation}">
+<xacro:unless value="${simulation}">
+  <ros2_control name="Actuator_${bl_label}" type="actuator">
+    <xacro:if value="${simulation}">
+      <hardware>
+        <plugin>gazebo_ros2_control/GazeboSystem</plugin>
+      </hardware>
+    </xacro:if>
+    <xacro:unless value="${simulation}">
+      <hardware>
+        <plugin>terrestrial_robot/BDC_LM298_SystemHardware</plugin>
+        <param name="pwm_freq">1000</param>
+        <param name="forward_pin">5</param>
+        <param name="backward_pin">6</param>
+        <param name="rpm">100</param>
+      </hardware>
+    </xacro:unless>
+    <joint name="Joint_${bl_label}">
+      <command_interface name="velocity" />
+      <state_interface name="velocity" />
+    </joint>
+  </ros2_control>
+  <ros2_control name="Actuator_${br_label}" type="actuator">
+    <xacro:if value="${simulation}">
+      <hardware>
+        <plugin>gazebo_ros2_control/GazeboSystem</plugin>
+      </hardware>
+    </xacro:if>
+    <xacro:unless value="${simulation}">
+      <hardware>
+        <plugin>terrestrial_robot/BDC_LM298_SystemHardware</plugin>
+        <param name="pwm_freq">1000</param>
+        <param name="forward_pin">12</param>
+        <param name="backward_pin">16</param>
+        <param name="rpm">10</param>
+      </hardware>
+    </xacro:unless>
+    <joint name="Joint_${br_label}">
+      <command_interface name="velocity" />
+      <state_interface name="velocity" />
+    </joint>
+  </ros2_control>
+  <ros2_control name="Actuator_${fr_label}" type="actuator">
+    <xacro:if value="${simulation}">
+      <hardware>
+        <plugin>gazebo_ros2_control/GazeboSystem</plugin>
+      </hardware>
+    </xacro:if>
+    <xacro:unless value="${simulation}">
+      <hardware>
+        <plugin>terrestrial_robot/BDC_LM298_SystemHardware</plugin>
+        <param name="pwm_freq">1000</param>
+        <param name="forward_pin">23</param>
+        <param name="backward_pin">24</param>
+        <param name="rpm">100</param>
+      </hardware>
+    </xacro:unless>
+    <joint name="Joint_${fr_label}">
+      <command_interface name="velocity" />
+      <state_interface name="velocity" />
+    </joint>
+  </ros2_control>
+  <ros2_control name="Actuator_${fl_label}" type="actuator">
+    <xacro:if value="${simulation}">
+      <hardware>
+        <plugin>gazebo_ros2_control/GazeboSystem</plugin>
+      </hardware>
+    </xacro:if>
+    <xacro:unless value="${simulation}">
+      <hardware>
+        <plugin>terrestrial_robot/BDC_LM298_SystemHardware</plugin>
+        <param name="pwm_freq">1000</param>
+        <param name="forward_pin">27</param>
+        <param name="backward_pin">22</param>
+        <param name="rpm">1000</param>
+      </hardware>
+    </xacro:unless>
+    <joint name="Joint_${fl_label}">
+      <command_interface name="velocity" />
+      <state_interface name="velocity" />
+    </joint>
+  </ros2_control>
+</xacro:unless>
+<xacro:if value="${simulation}">
+  <ros2_control name="GazeboSystem" type="system">
     <hardware>
       <plugin>gazebo_ros2_control/GazeboSystem</plugin>
     </hardware>
-  </xacro:if>
-  <xacro:unless value="${simulation}">
-    <hardware>
-      <plugin>terrestrial_robot/BDC_LM298_SystemHardware</plugin>
-      <param name="pwm_freq">1000</param>
-      <param name="forward_pin">5</param>
-      <param name="backward_pin">6</param>
-      <param name="rpm">100</param>
-    </hardware>
-  </xacro:unless>
-  <joint name="Joint_${bl_label}">
-    <command_interface name="velocity" />
-    <state_interface name="velocity" />
-  </joint>
-</ros2_control>
-<ros2_control name="Actuator_${br_label}" type="actuator">
-  <xacro:if value="${simulation}">
-    <hardware>
-      <plugin>gazebo_ros2_control/GazeboSystem</plugin>
-    </hardware>
-  </xacro:if>
-  <xacro:unless value="${simulation}">
-    <hardware>
-      <plugin>terrestrial_robot/BDC_LM298_SystemHardware</plugin>
-      <param name="pwm_freq">1000</param>
-      <param name="forward_pin">12</param>
-      <param name="backward_pin">16</param>
-      <param name="rpm">10</param>
-    </hardware>
-  </xacro:unless>
-  <joint name="Joint_${br_label}">
-    <command_interface name="velocity" />
-    <state_interface name="velocity" />
-  </joint>
-</ros2_control>
-<ros2_control name="Actuator_${fr_label}" type="actuator">
-  <xacro:if value="${simulation}">
-    <hardware>
-      <plugin>gazebo_ros2_control/GazeboSystem</plugin>
-    </hardware>
-  </xacro:if>
-  <xacro:unless value="${simulation}">
-    <hardware>
-      <plugin>terrestrial_robot/BDC_LM298_SystemHardware</plugin>
-      <param name="pwm_freq">1000</param>
-      <param name="forward_pin">23</param>
-      <param name="backward_pin">24</param>
-      <param name="rpm">100</param>
-    </hardware>
-  </xacro:unless>
-  <joint name="Joint_${fr_label}">
-    <command_interface name="velocity" />
-    <state_interface name="velocity" />
-  </joint>
-</ros2_control>
-<ros2_control name="Actuator_${fl_label}" type="actuator">
-  <xacro:if value="${simulation}">
-    <hardware>
-      <plugin>gazebo_ros2_control/GazeboSystem</plugin>
-    </hardware>
-  </xacro:if>
-  <xacro:unless value="${simulation}">
-    <hardware>
-      <plugin>terrestrial_robot/BDC_LM298_SystemHardware</plugin>
-      <param name="pwm_freq">1000</param>
-      <param name="forward_pin">27</param>
-      <param name="backward_pin">22</param>
-      <param name="rpm">1000</param>
-    </hardware>
-  </xacro:unless>
-  <joint name="Joint_${fl_label}">
-    <command_interface name="velocity" />
-    <state_interface name="velocity" />
-  </joint>
-</ros2_control>
+    <joint name="Joint_${bl_label}">
+      <command_interface name="velocity" />
+      <state_interface name="velocity" />
+    </joint>
+    <joint name="Joint_${br_label}">
+      <command_interface name="velocity" />
+      <state_interface name="velocity" />
+    </joint>
+    <joint name="Joint_${fr_label}">
+      <command_interface name="velocity" />
+      <state_interface name="velocity" />
+    </joint>
+    <joint name="Joint_${fl_label}">
+      <command_interface name="velocity" />
+      <state_interface name="velocity" />
+    </joint>
+  </ros2_control>
+</xacro:if>
 <gazebo>
     <plugin filename="libgazebo_ros2_control.so" name="gazebo_ros2_control">
       <robot_param>robot_description</robot_param>
       <robot_param_node>robot_state_publisher</robot_param_node>
-      <parameters>$(find terrestrial_robot)/config/controller.yaml</parameters>
+      <parameters>$(find terrestrial_robot)/config/sim_controller.yaml</parameters>
     </plugin>
 </gazebo>
